File: ARM.kicad_sch (KiCad schematic)
At the start: 52 parts, among them J1 AVR-ISP-6, SW1 4-1437565-9, U1 DSPIC33FJ64MC802-xSP, U2 AMS1117-3.3v, X1 AVR-ICSP, X2 AVR-ICSP, X3 AVR-ICSP, Y1 Crystal hc49 20Mhz

Commit message: push files
Parts:
- removed C10, C11, C9: 470UF 10V baja ESR, Capacitor_THT:C_Radial_D8.0mm_H7.0mm_P3.50mm, symbol Device:C
- removed C12: 2200 µF / 10 V baja ESR, Capacitor_THT:C_Radial_D10.0mm_H12.5mm_P5.00mm, symbol Device:C
- removed C19, C20: 0.1UF, Capacitor_SMD:C_0603_1608Metric, symbol Device:C
- removed C23: C, Capacitor_SMD:C_Elec_6.3x5.8, symbol Device:C
- removed C4, C5: CERAMIC-10UF-25V-10_-X5R_1206_, CERAMIC-10UF-25V-10_-X5R_1206_:C1206, symbol CERAMIC-10UF-25V-10_-X5R_1206_:CERAMIC-10UF-25V-10_-X5R_1206_
- removed C6: CERAMIC-1UF-25V-10_-X5R_1206_, CERAMIC-10UF-25V-10_-X5R_1206_:C1206, symbol CERAMIC-10UF-25V-10_-X5R_1206_:CERAMIC-10UF-25V-10_-X5R_1206_
- removed C7: CERAMIC-4,7UF-25V-10_-X5R_1206_, CERAMIC-10UF-25V-10_-X5R_1206_:C1206, symbol CERAMIC-10UF-25V-10_-X5R_1206_:CERAMIC-10UF-25V-10_-X5R_1206_
- removed C8: CERAMIC-22UF-25V-10_-X5R_1206_, CERAMIC-10UF-25V-10_-X5R_1206_:C1206, symbol CERAMIC-10UF-25V-10_-X5R_1206_:CERAMIC-10UF-25V-10_-X5R_1206_
- removed F1: 1812L300_24SLER, Polyfuse1812L300_24SLER:FUSSC324X455X250-2N, symbol 1812L300_24SLER:1812L300_24SLER
- removed F2: 0ZCF0030FF2C, ul_0ZCF0030FF2C:0ZCF_BEL, symbol 2025-08-20_01-47-34:0ZCF0030FF2C
- removed J1: AVR-ISP-6, Connector_IDC:IDC-Header_2x03_P2.54mm_Vertical, symbol Connector:AVR-ISP-6
- removed L1: B82462G4103M000, IND_EPCOS_B82462G4_EPC, symbol 2025-08-20_19-40-59:B82462G4103M000
- removed U1: DSPIC33FJ64MC802-xSP, Package_DIP:DIP-28_W7.62mm_Socket_LongPads, symbol DSP_Microchip_DSPIC33:DSPIC33FJ64MC802-xSP
- removed X1, X2, X3: AVR-ICSP, AVR-ICSP:ICSP-2X03-2.54, symbol AVR-ICSP:AVR-ICSP
- added C1: 2200µF 25v baja ESR, Capacitor_SMD:CP_Elec_10x10.5, symbol Device:C_Polarized
- added C12: 47µF 16v, Capacitor_SMD:CP_Elec_8x6.2, symbol Device:C_Polarized
- added C14: 10µF 16v, Capacitor_SMD:C_1206_3216Metric, symbol Device:C
- added C15: 0.1 µF 16v, Capacitor_SMD:C_0805_2012Metric, symbol Device:C
- added C16, C17: 22pF 16v, Capacitor_SMD:C_0805_2012Metric_Pad1.18x1.45mm_HandSolder, symbol Device:C
- added C2: 4.7UF 16v, Capacitor_SMD:CP_Elec_8x10.5, symbol Device:C_Polarized
- added C24: 1UF-16V, Capacitor_SMD:C_1210_3225Metric_Pad1.33x2.70mm_HandSolder, symbol Device:C
- added C25: 4,7UF-16V, Capacitor_SMD:C_1210_3225Metric_Pad1.33x2.70mm_HandSolder, symbol Device:C
- added C26, C28, C29: 10UF-16V, Capacitor_SMD:C_1210_3225Metric_Pad1.33x2.70mm_HandSolder, symbol Device:C
- added C27: 22UF-16V, Capacitor_SMD:C_1210_3225Metric_Pad1.33x2.70mm_HandSolder, symbol Device:C
- added C3, C4, C5: 470UF 16V baja ESR, Capacitor_SMD:CP_Elec_8x6.2, symbol Device:C_Polarized
- added C30: 0.1µF 16V, Capacitor_SMD:C_0805_2012Metric_Pad1.18x1.45mm_HandSolder, symbol Device:C
- added D6: LED White, LED_SMD:LED_0805_2012Metric_Pad1.15x1.40mm_HandSolder, symbol Device:LED
- added D7: LED Yellow, LED_SMD:LED_0805_2012Metric_Pad1.15x1.40mm_HandSolder, symbol Device:LED
- added D8: LED Orange, LED_SMD:LED_0805_2012Metric_Pad1.15x1.40mm_HandSolder, symbol Device:LED
- added F1: 500mA, 1812L110_24DR:FUSM4632X200N, symbol 1812L110_24DR:1812L110_24DR
- added F2: 3A, ul_PTS18126V300:FUSE_PTS18126_COB, symbol 2025-08-30_23-17-27:PTS18126V300
- added J1: USB_OTG, Connector_USB:USB_Mini-B_Lumberg_2486_01_Horizontal, symbol Connector:USB_OTG
- added J14: Conn_01x07_Socket, Connector_PinHeader_2.54mm:PinHeader_1x07_P2.54mm_Vertical_SMD_Pin1Left, symbol Connector:Conn_01x07_Socket
- added J2: USB_C_PowerOnly_6P +5v, Connector_USB:USB_C_Receptacle_GCT_USB4135-GF-A_6P_TopMnt_Horizontal, symbol Connector:USB_C_Receptacle_PowerOnly_6P
- added J3, J4, J5: G823MB06221KYEU, G823MB06221KYEU:AMPHENOL_G823MB06221KYEU, symbol G823MB06221KYEU:G823MB06221KYEU
- added J8: Conn_01x04_Socket, Connector_PinSocket_2.54mm:PinSocket_1x04_P2.54mm_Vertical_SMD_Pin1Left, symbol Connector:Conn_01x04_Socket
- added J9: Conn_01x02_Socket, Connector_PinHeader_2.54mm:PinHeader_1x02_P2.54mm_Vertical, symbol Connector:Conn_01x02_Socket
- added L1: L_Small, Inductor_SMD:L_TDK_SLF6045, symbol Device:L_Small
- added R14, R15, R16, R17: 10KΩ 1%, Resistor_SMD:R_0805_2012Metric_Pad1.20x1.40mm_HandSolder, symbol Device:R
- added R19, R6: 330Ω 1%, Resistor_SMD:R_0805_2012Metric_Pad1.20x1.40mm_HandSolder, symbol Device:R
- added R20, R21, R23, R24: 33Ω 1%, Resistor_SMD:R_0805_2012Metric_Pad1.20x1.40mm_HandSolder, symbol Device:R
- added R22, R25: 10 kΩ 1%, Resistor_SMD:R_0805_2012Metric_Pad1.20x1.40mm_HandSolder, symbol Device:R
- added R9: 220Ω 1%, Resistor_SMD:R_0805_2012Metric_Pad1.20x1.40mm_HandSolder, symbol Device:R
- added U1: ATMEGA328-PU, Package_DIP:DIP-28_W7.62mm_Socket_LongPads, symbol ATMEGA328-PU:ATMEGA328-PU
- added U3: CH340G, Package_SO:SOIC-16_3.9x9.9mm_P1.27mm, symbol Interface_USB:CH340G
- added Y2: 12Mhz, Crystal:Crystal_SMD_HC49-SD, symbol Device:Crystal
- C10: renamed from C22; value 0.1UF -> 0.1UF 16v
- C11: renamed from C21; value 0.1UF -> 0.1UF 16v
- C7: renamed from C3; value 100nF -> 100nF 16v
- C8: renamed from C2; value 22pF -> 22pF 16v
- C9: renamed from C1; value 22pF -> 22pF 16v
- D3: value LED -> LED Red
- D4: value LED -> LED Green
- D5: renamed from D2; value LED -> LED Blue
- FB1: value FerriteBead -> Ferrite 100MHz 600Ω 2A
- R1: value 10k -> 10 kΩ 1%
- R10, R11, R8: value 10KΩ -> 220Ω 1%; footprint Resistor_SMD:R_0805_2012Metric -> Resistor_SMD:R_0805_2012Metric_Pad1.20x1.40mm_HandSolder
- R12: renamed from R6; value 220Ω -> 220Ω 1%; footprint Resistor_SMD:R_0805_2012Metric -> Resistor_SMD:R_0805_2012Metric_Pad1.20x1.40mm_HandSolder
- R13: renamed from R9; value 10KΩ -> 10KΩ 1%; footprint Resistor_SMD:R_0805_2012Metric -> Resistor_SMD:R_0805_2012Metric_Pad1.20x1.40mm_HandSolder
- R18: renamed from R12; value 10KΩ -> 10KΩ 1%; footprint Resistor_SMD:R_0805_2012Metric -> Resistor_SMD:R_0805_2012Metric_Pad1.20x1.40mm_HandSolder
- R2: value 300ohm -> 330Ω 1%
- R3, R4, R5: value 220Ω -> 330Ω 1%; footprint Resistor_SMD:R_0805_2012Metric -> Resistor_SMD:R_0805_2012Metric_Pad1.20x1.40mm_HandSolder
- R7: value 220Ω -> 220Ω 1%; footprint Resistor_SMD:R_0805_2012Metric -> Resistor_SMD:R_0805_2012Metric_Pad1.20x1.40mm_HandSolder
- Y1: value Crystal hc49 20Mhz -> Crystal 20Mhz
- renumbered C17 to C19, C16 to C20, C15 to C21, C14 to C22, C13 to C23, D5 to D2
Connections:
- net at R5.1: now also D6.2 (A)
- net +5vSe: now reaches R5.2
- net +5vSe: now also C10.1, C11.1, C18.2, C19.1, C20.1, C21.1, C22.1, C23.2, C7.1, D1.1 (K), R1.1, R4.2, C1.1, C12.1, C14.2, C15.2, C24.1, C25.2, C26.2, C27.2, C3.1, C4.1, C5.1, F2.1, J1.1 (VBUS), J3.3, J3.4, J4.3, J4.4, J5.3, J5.4, L1.2, R22.1, R25.1, U1.20 (AVCC), U1.7 (VCC), U3.16 (VCC)
- net GND: now reaches C7.2
- net GND: now also C10.2, C11.2, C18.1, C19.2, C20.2, C21.2, C22.2, C23.1, C8.2, C9.1, D2.1 (A1), D3.1 (K), D4.1 (K), D5.1 (K), SW1.1, SW1.2, U2.1 (GND), C1.2, C12.2, C14.1, C15.1, C16.1, C17.1, C2.2, C24.2, C25.1, C26.1, C27.1, C28.2, C29.2, C3.2, C30.2, C4.2, C5.2, D6.1 (K), D7.1 (K), D8.1 (K), J1.5 (GND), J1.6 (Shield), J2.A12 (GND), J2.B12 (GND), J2.S1 (SHIELD), J3.1, J3.2, J4.1, J4.2, J5.1, J5.2, J9.1 (Pin_1), U1.22 (GND__1), U1.8 (GND), U3.1 (GND)
- net at Y1.1: now also C9.2, U1.9 (PB6(PCINT6/XTAL1/TOSC1))
- net at Y1.2: now also C8.1, U1.10 (PB7(PCINT7/XTAL2/TOSC2))
- net +5vTo3,3v: now reaches D1.2 (A)
- net +5vTo3,3v: now also D2.2 (A2), U2.3 (VI), C28.1, F1.2
- net at R18.1: now also U1.28 (PC5(ADC5/SCL/PCINT13))
- net at R18.2: now also J14.6 (Pin_6)
- net at R2.1: now also D5.2 (A)
- net at R2.2: now also U1.15 (PB1(OC1A/PCINT1))
- net at R1.2: now also SW1.3, SW1.4, U1.1 (PC6(PCINT14/~{RESET}))
- net at R10.1: now also U1.11 (PD5(PCINT21/OC0B/T1))
- net S4: now reaches R10.2
- net S4: now also J4.5
- net at R11.1: now also U1.12 (PD6(PCINT22/OC0A/AIN0))
- net S5: now reaches R11.2
- net S5: now also J5.6
- net at D4.2 (A): now also R3.1
- net at D3.2 (A): now also R4.1
- net at R8.1: now also U1.5 (PD3(PCINT19/OC2B/INT1))
- net S2: now reaches R8.2
- net S2: now also J3.5
- net at R12.1: now also U1.13 (PD7(PCINT23/AIN1))
- net S6: now reaches R12.2
- net S6: now also J5.5
- net at FB1.1: now also U2.2 (VO), C29.1
- net 3,3v: now reaches FB1.2
- net 3,3v: now also C30.1, J14.7 (Pin_7)
- net at R3.2: now also U1.14 (PB0(PCINT0/CLKO/ICP1))
- net at R13.1: now also U1.23 (PC0(ADC0/PCINT8))
- net at R13.2: now also J14.1 (Pin_1)
- net at R7.1: now also U1.4 (PD2(PCINT18/INT0))
- net S1: now reaches R7.2
- net S1: now also J3.6
- new net: J1.2 (D-), U3.6 (UD-)
- new net: J1.3 (D+), U3.5 (UD+)
- new net: R24.2, R25.2, U1.16 (PB2(~{SS}/OC1B/PCINT2))
- new net: D7.2 (A), R6.1
- new net: R21.2, R22.2, U1.18 (PB4(MISO/PCINT4))
- new net: D8.2 (A), R19.1
- new net: R23.2, U1.19 (PB5(SCK/PCINT5))
- new net: C17.2, U3.8 (XO), Y2.1
- new net: C16.2, U3.7 (XI), Y2.2
- new net: J14.2 (Pin_2), R14.2
- new net: J14.3 (Pin_3), R15.2
- new net: J14.4 (Pin_4), R16.2
- new net: J14.5 (Pin_5), R17.2
- new net: C2.1, F2.2, L1.1
- new net: R16.1, U1.26 (PC3(ADC3/PCINT11))
- new net: R15.1, U1.25 (PC2(ADC2/PCINT10))
- new net: R17.1, U1.27 (PC4(ADC4/SDA/PCINT12))
- new net: R20.2, U1.17 (PB3(MOSI/OC2A/PCINT3))
- new net: R14.1, U1.24 (PC1(ADC1/PCINT9))
- new net: R9.1, U1.6 (PD4(PCINT20/XCK/T0))
- new net +5vE: F1.1, J2.A9 (VBUS), J2.B9 (VBUS), J9.2 (Pin_2)
- new net ISP1: J8.1 (Pin_1), R20.1
- new net ISP2: J8.2 (Pin_2), R21.1
- new net ISP3: J8.3 (Pin_3), R23.1
- new net ISP4: J8.4 (Pin_4), R24.1
- new net S3: J4.6, R9.2
- new net USB_RX: R6.2, U1.2 (PD0(PCINT16/RXD)), U3.2 (TXD)
- new net USB_TX: R19.2, U1.3 (PD1(PCINT17/TXD)), U3.3 (RXD)
- no-connect marks 0 -> 12
Other:
- note added: "3 Jumpers de conexion dobles para 6 servos"
- note added: "Modulo de Energia"
- note added: "Modulo de control (Principal)"
- note added: "Modulo regulador 3,3v"
- note added: "Módulo de Comunicación USB (USB-UART)"
- moved on the sheet: C10, C11, C18, C19, C20, C21, C22, C23, C7, C8, C9, D1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

Commit message: mistake
Parts:
- removed C1: 2200µF 25v baja ESR, Capacitor_SMD:CP_Elec_10x10.5, symbol Device:C_Polarized
- removed C10, C11: 0.1UF 16v, Capacitor_SMD:C_0603_1608Metric, symbol Device:C
- removed C12: 47µF 16v, Capacitor_SMD:CP_Elec_8x6.2, symbol Device:C_Polarized
- removed C14: 10µF 16v, Capacitor_SMD:C_1206_3216Metric, symbol Device:C
- removed C15: 0.1 µF 16v, Capacitor_SMD:C_0805_2012Metric, symbol Device:C
- removed C16, C17, C8, C9: 22pF 16v, Capacitor_SMD:C_0805_2012Metric_Pad1.18x1.45mm_HandSolder, symbol Device:C
- removed C18, C19, C20, C21, C22, C23: 100NF, Capacitor_SMD:C_0805_2012Metric, symbol Device:C
- removed C2: 4.7UF 16v, Capacitor_SMD:CP_Elec_8x10.5, symbol Device:C_Polarized
- removed C24: 1UF-16V, Capacitor_SMD:C_1210_3225Metric_Pad1.33x2.70mm_HandSolder, symbol Device:C
- removed C25: 4,7UF-16V, Capacitor_SMD:C_1210_3225Metric_Pad1.33x2.70mm_HandSolder, symbol Device:C
- removed C26, C28, C29: 10UF-16V, Capacitor_SMD:C_1210_3225Metric_Pad1.33x2.70mm_HandSolder, symbol Device:C
- removed C27: 22UF-16V, Capacitor_SMD:C_1210_3225Metric_Pad1.33x2.70mm_HandSolder, symbol Device:C
- removed C3, C4, C5: 470UF 16V baja ESR, Capacitor_SMD:CP_Elec_8x6.2, symbol Device:C_Polarized
- removed C30: 0.1µF 16V, Capacitor_SMD:C_0805_2012Metric_Pad1.18x1.45mm_HandSolder, symbol Device:C
- removed C7: 100nF 16v, Capacitor_SMD:C_0805_2012Metric_Pad1.18x1.45mm_HandSolder, symbol Device:C
- removed D1: SS14, Diode_SMD:D_SMA, symbol Diode:SS14
- removed D2: D_TVS 9V SMBJ12A, Diode_SMD:D_SMB, symbol Device:D_TVS
- removed D3: LED Red, LED_SMD:LED_0805_2012Metric, symbol Device:LED
- removed D4: LED Green, LED_SMD:LED_0805_2012Metric, symbol Device:LED
- removed D5: LED Blue, LED_SMD:LED_0805_2012Metric_Pad1.15x1.40mm_HandSolder, symbol Device:LED
- removed D6: LED White, LED_SMD:LED_0805_2012Metric_Pad1.15x1.40mm_HandSolder, symbol Device:LED
- removed D7: LED Yellow, LED_SMD:LED_0805_2012Metric_Pad1.15x1.40mm_HandSolder, symbol Device:LED
- removed D8: LED Orange, LED_SMD:LED_0805_2012Metric_Pad1.15x1.40mm_HandSolder, symbol Device:LED
- removed F1: 500mA, 1812L110_24DR:FUSM4632X200N, symbol 1812L110_24DR:1812L110_24DR
- removed F2: 3A, ul_PTS18126V300:FUSE_PTS18126_COB, symbol 2025-08-30_23-17-27:PTS18126V300
- removed FB1: Ferrite 100MHz 600Ω 2A, Inductor_SMD:L_0805_2012Metric_Pad1.15x1.40mm_HandSolder, symbol Device:FerriteBead
- removed J1: USB_OTG, Connector_USB:USB_Mini-B_Lumberg_2486_01_Horizontal, symbol Connector:USB_OTG
- removed J14: Conn_01x07_Socket, Connector_PinHeader_2.54mm:PinHeader_1x07_P2.54mm_Vertical_SMD_Pin1Left, symbol Connector:Conn_01x07_Socket
- removed J2: USB_C_PowerOnly_6P +5v, Connector_USB:USB_C_Receptacle_GCT_USB4135-GF-A_6P_TopMnt_Horizontal, symbol Connector:USB_C_Receptacle_PowerOnly_6P
- removed J3, J4, J5: G823MB06221KYEU, G823MB06221KYEU:AMPHENOL_G823MB06221KYEU, symbol G823MB06221KYEU:G823MB06221KYEU
- removed J8: Conn_01x04_Socket, Connector_PinSocket_2.54mm:PinSocket_1x04_P2.54mm_Vertical_SMD_Pin1Left, symbol Connector:Conn_01x04_Socket
- removed J9: Conn_01x02_Socket, Connector_PinHeader_2.54mm:PinHeader_1x02_P2.54mm_Vertical, symbol Connector:Conn_01x02_Socket
- removed L1: L_Small, Inductor_SMD:L_TDK_SLF6045, symbol Device:L_Small
- removed R1, R22, R25: 10 kΩ 1%, Resistor_SMD:R_0805_2012Metric_Pad1.20x1.40mm_HandSolder, symbol Device:R
- removed R10, R11, R12, R7, R8, R9: 220Ω 1%, Resistor_SMD:R_0805_2012Metric_Pad1.20x1.40mm_HandSolder, symbol Device:R
- removed R13, R14, R15, R16, R17, R18: 10KΩ 1%, Resistor_SMD:R_0805_2012Metric_Pad1.20x1.40mm_HandSolder, symbol Device:R
- removed R19, R2, R3, R4, R5, R6: 330Ω 1%, Resistor_SMD:R_0805_2012Metric_Pad1.20x1.40mm_HandSolder, symbol Device:R
- removed R20, R21, R23, R24: 33Ω 1%, Resistor_SMD:R_0805_2012Metric_Pad1.20x1.40mm_HandSolder, symbol Device:R
- removed SW1: 4-1437565-9, 4-1437565-9:TE_4-1437565-9, symbol 4-1437565-9:4-1437565-9
- removed U1: ATMEGA328-PU, Package_DIP:DIP-28_W7.62mm_Socket_LongPads, symbol ATMEGA328-PU:ATMEGA328-PU
- removed U2: AMS1117-3.3v, Package_TO_SOT_SMD:SOT-223-3_TabPin2, symbol Regulator_Linear:AMS1117-5.0
- removed U3: CH340G, Package_SO:SOIC-16_3.9x9.9mm_P1.27mm, symbol Interface_USB:CH340G
- removed Y1: Crystal 20Mhz, Crystal:Crystal_SMD_HC49-SD, symbol Device:Crystal
- removed Y2: 12Mhz, Crystal:Crystal_SMD_HC49-SD, symbol Device:Crystal
Connections:
- no-connect marks 12 -> 0
Other:
- note removed: "3 Jumpers de conexion dobles para 6 servos"
- note removed: "Modulo de Energia"
- note removed: "Modulo de control (Principal)"
- note removed: "Modulo regulador 3,3v"
- note removed: "Módulo de Comunicación USB (USB-UART)"

Commit message: Revert "mistake"
This reverts commit 8728f3de92bb642d3a5581e7387178a88eb5d2a4.
Parts:
- added C1: 2200µF 25v baja ESR, Capacitor_SMD:CP_Elec_10x10.5, symbol Device:C_Polarized
- added C10, C11: 0.1UF 16v, Capacitor_SMD:C_0603_1608Metric, symbol Device:C
- added C12: 47µF 16v, Capacitor_SMD:CP_Elec_8x6.2, symbol Device:C_Polarized
- added C14: 10µF 16v, Capacitor_SMD:C_1206_3216Metric, symbol Device:C
- added C15: 0.1 µF 16v, Capacitor_SMD:C_0805_2012Metric, symbol Device:C
- added C16, C17, C8, C9: 22pF 16v, Capacitor_SMD:C_0805_2012Metric_Pad1.18x1.45mm_HandSolder, symbol Device:C
- added C18, C19, C20, C21, C22, C23: 100NF, Capacitor_SMD:C_0805_2012Metric, symbol Device:C
- added C2: 4.7UF 16v, Capacitor_SMD:CP_Elec_8x10.5, symbol Device:C_Polarized
- added C24: 1UF-16V, Capacitor_SMD:C_1210_3225Metric_Pad1.33x2.70mm_HandSolder, symbol Device:C
- added C25: 4,7UF-16V, Capacitor_SMD:C_1210_3225Metric_Pad1.33x2.70mm_HandSolder, symbol Device:C
- added C26, C28, C29: 10UF-16V, Capacitor_SMD:C_1210_3225Metric_Pad1.33x2.70mm_HandSolder, symbol Device:C
- added C27: 22UF-16V, Capacitor_SMD:C_1210_3225Metric_Pad1.33x2.70mm_HandSolder, symbol Device:C
- added C3, C4, C5: 470UF 16V baja ESR, Capacitor_SMD:CP_Elec_8x6.2, symbol Device:C_Polarized
- added C30: 0.1µF 16V, Capacitor_SMD:C_0805_2012Metric_Pad1.18x1.45mm_HandSolder, symbol Device:C
- added C7: 100nF 16v, Capacitor_SMD:C_0805_2012Metric_Pad1.18x1.45mm_HandSolder, symbol Device:C
- added D1: SS14, Diode_SMD:D_SMA, symbol Diode:SS14
- added D2: D_TVS 9V SMBJ12A, Diode_SMD:D_SMB, symbol Device:D_TVS
- added D3: LED Red, LED_SMD:LED_0805_2012Metric, symbol Device:LED
- added D4: LED Green, LED_SMD:LED_0805_2012Metric, symbol Device:LED
- added D5: LED Blue, LED_SMD:LED_0805_2012Metric_Pad1.15x1.40mm_HandSolder, symbol Device:LED
- added D6: LED White, LED_SMD:LED_0805_2012Metric_Pad1.15x1.40mm_HandSolder, symbol Device:LED
- added D7: LED Yellow, LED_SMD:LED_0805_2012Metric_Pad1.15x1.40mm_HandSolder, symbol Device:LED
- added D8: LED Orange, LED_SMD:LED_0805_2012Metric_Pad1.15x1.40mm_HandSolder, symbol Device:LED
- added F1: 500mA, 1812L110_24DR:FUSM4632X200N, symbol 1812L110_24DR:1812L110_24DR
- added F2: 3A, ul_PTS18126V300:FUSE_PTS18126_COB, symbol 2025-08-30_23-17-27:PTS18126V300
- added FB1: Ferrite 100MHz 600Ω 2A, Inductor_SMD:L_0805_2012Metric_Pad1.15x1.40mm_HandSolder, symbol Device:FerriteBead
- added J1: USB_OTG, Connector_USB:USB_Mini-B_Lumberg_2486_01_Horizontal, symbol Connector:USB_OTG
- added J14: Conn_01x07_Socket, Connector_PinHeader_2.54mm:PinHeader_1x07_P2.54mm_Vertical_SMD_Pin1Left, symbol Connector:Conn_01x07_Socket
- added J2: USB_C_PowerOnly_6P +5v, Connector_USB:USB_C_Receptacle_GCT_USB4135-GF-A_6P_TopMnt_Horizontal, symbol Connector:USB_C_Receptacle_PowerOnly_6P
- added J3, J4, J5: G823MB06221KYEU, G823MB06221KYEU:AMPHENOL_G823MB06221KYEU, symbol G823MB06221KYEU:G823MB06221KYEU
- added J8: Conn_01x04_Socket, Connector_PinSocket_2.54mm:PinSocket_1x04_P2.54mm_Vertical_SMD_Pin1Left, symbol Connector:Conn_01x04_Socket
- added J9: Conn_01x02_Socket, Connector_PinHeader_2.54mm:PinHeader_1x02_P2.54mm_Vertical, symbol Connector:Conn_01x02_Socket
- added L1: L_Small, Inductor_SMD:L_TDK_SLF6045, symbol Device:L_Small
- added R1, R22, R25: 10 kΩ 1%, Resistor_SMD:R_0805_2012Metric_Pad1.20x1.40mm_HandSolder, symbol Device:R
- added R10, R11, R12, R7, R8, R9: 220Ω 1%, Resistor_SMD:R_0805_2012Metric_Pad1.20x1.40mm_HandSolder, symbol Device:R
- added R13, R14, R15, R16, R17, R18: 10KΩ 1%, Resistor_SMD:R_0805_2012Metric_Pad1.20x1.40mm_HandSolder, symbol Device:R
- added R19, R2, R3, R4, R5, R6: 330Ω 1%, Resistor_SMD:R_0805_2012Metric_Pad1.20x1.40mm_HandSolder, symbol Device:R
- added R20, R21, R23, R24: 33Ω 1%, Resistor_SMD:R_0805_2012Metric_Pad1.20x1.40mm_HandSolder, symbol Device:R
- added SW1: 4-1437565-9, 4-1437565-9:TE_4-1437565-9, symbol 4-1437565-9:4-1437565-9
- added U1: ATMEGA328-PU, Package_DIP:DIP-28_W7.62mm_Socket_LongPads, symbol ATMEGA328-PU:ATMEGA328-PU
- added U2: AMS1117-3.3v, Package_TO_SOT_SMD:SOT-223-3_TabPin2, symbol Regulator_Linear:AMS1117-5.0
- added U3: CH340G, Package_SO:SOIC-16_3.9x9.9mm_P1.27mm, symbol Interface_USB:CH340G
- added Y1: Crystal 20Mhz, Crystal:Crystal_SMD_HC49-SD, symbol Device:Crystal
- added Y2: 12Mhz, Crystal:Crystal_SMD_HC49-SD, symbol Device:Crystal
Connections:
- new net: J1.2 (D-), U3.6 (UD-)
- new net: J1.3 (D+), U3.5 (UD+)
- new net: R24.2, R25.2, U1.16 (PB2(~{SS}/OC1B/PCINT2))
- new net: D6.2 (A), R5.1
- new net: R1.2, SW1.3, SW1.4, U1.1 (PC6(PCINT14/~{RESET}))
- new net: C9.2, U1.9 (PB6(PCINT6/XTAL1/TOSC1)), Y1.1
- new net: C8.1, U1.10 (PB7(PCINT7/XTAL2/TOSC2)), Y1.2
- new net: D7.2 (A), R6.1
- new net: R21.2, R22.2, U1.18 (PB4(MISO/PCINT4))
- new net: D8.2 (A), R19.1
- new net: R23.2, U1.19 (PB5(SCK/PCINT5))
- new net: C17.2, U3.8 (XO), Y2.1
- new net: C16.2, U3.7 (XI), Y2.2
- new net: J14.1 (Pin_1), R13.2
- new net: J14.2 (Pin_2), R14.2
- new net: J14.3 (Pin_3), R15.2
- new net: J14.4 (Pin_4), R16.2
- new net: J14.5 (Pin_5), R17.2
- new net: J14.6 (Pin_6), R18.2
- new net: C2.1, F2.2, L1.1
- new net: R16.1, U1.26 (PC3(ADC3/PCINT11))
- new net: R18.1, U1.28 (PC5(ADC5/SCL/PCINT13))
- new net: D5.2 (A), R2.1
- new net: R2.2, U1.15 (PB1(OC1A/PCINT1))
- new net: R15.1, U1.25 (PC2(ADC2/PCINT10))
- new net: R10.1, U1.11 (PD5(PCINT21/OC0B/T1))
- new net: R17.1, U1.27 (PC4(ADC4/SDA/PCINT12))
- new net: R11.1, U1.12 (PD6(PCINT22/OC0A/AIN0))
- new net: D4.2 (A), R3.1
- new net: D3.2 (A), R4.1
- new net: R8.1, U1.5 (PD3(PCINT19/OC2B/INT1))
- new net: R12.1, U1.13 (PD7(PCINT23/AIN1))
- new net: R3.2, U1.14 (PB0(PCINT0/CLKO/ICP1))
- new net: R20.2, U1.17 (PB3(MOSI/OC2A/PCINT3))
- new net: R13.1, U1.23 (PC0(ADC0/PCINT8))
- new net: R14.1, U1.24 (PC1(ADC1/PCINT9))
- new net: R7.1, U1.4 (PD2(PCINT18/INT0))
- new net: R9.1, U1.6 (PD4(PCINT20/XCK/T0))
- new net: C29.1, FB1.1, U2.2 (VO)
- new net +5vE: F1.1, J2.A9 (VBUS), J2.B9 (VBUS), J9.2 (Pin_2)
- new net +5vSe: C1.1, C10.1, C11.1, C12.1, C14.2, C15.2, C18.2, C19.1, C20.1, C21.1, C22.1, C23.2, C24.1, C25.2, C26.2, C27.2, C3.1, C4.1, C5.1, C7.1, D1.1 (K), F2.1, J1.1 (VBUS), J3.3, J3.4, J4.3, J4.4, J5.3, J5.4, L1.2, R1.1, R22.1, R25.1, R4.2, R5.2, U1.20 (AVCC), U1.7 (VCC), U3.16 (VCC)
- new net +5vTo3,3v: C28.1, D1.2 (A), D2.2 (A2), F1.2, U2.3 (VI)
- new net 3,3v: C30.1, FB1.2, J14.7 (Pin_7)
- new net GND: C1.2, C10.2, C11.2, C12.2, C14.1, C15.1, C16.1, C17.1, C18.1, C19.2, C2.2, C20.2, C21.2, C22.2, C23.1, C24.2, C25.1, C26.1, C27.1, C28.2, C29.2, C3.2, C30.2, C4.2, C5.2, C7.2, C8.2, C9.1, D2.1 (A1), D3.1 (K), D4.1 (K), D5.1 (K), D6.1 (K), D7.1 (K), D8.1 (K), J1.5 (GND), J1.6 (Shield), J2.A12 (GND), J2.B12 (GND), J2.S1 (SHIELD), J3.1, J3.2, J4.1, J4.2, J5.1, J5.2, J9.1 (Pin_1), SW1.1, SW1.2, U1.22 (GND__1), U1.8 (GND), U2.1 (GND), U3.1 (GND)
- new net ISP1: J8.1 (Pin_1), R20.1
- new net ISP2: J8.2 (Pin_2), R21.1
- new net ISP3: J8.3 (Pin_3), R23.1
- new net ISP4: J8.4 (Pin_4), R24.1
- new net S1: J3.6, R7.2
- new net S2: J3.5, R8.2
- new net S3: J4.6, R9.2
- new net S4: J4.5, R10.2
- new net S5: J5.6, R11.2
- new net S6: J5.5, R12.2
- new net USB_RX: R6.2, U1.2 (PD0(PCINT16/RXD)), U3.2 (TXD)
- new net USB_TX: R19.2, U1.3 (PD1(PCINT17/TXD)), U3.3 (RXD)
- no-connect marks 0 -> 12
Other:
- note added: "3 Jumpers de conexion dobles para 6 servos"
- note added: "Modulo de Energia"
- note added: "Modulo de control (Principal)"
- note added: "Modulo regulador 3,3v"
- note added: "Módulo de Comunicación USB (USB-UART)"
